File: circuits/led-controller.sch (KiCad schematic (older format))
At the start: 24 parts

Commit message: adding sheets
Parts:
- removed C? (x4): C_1uF, Capacitor_SMD:C_0603_1608Metric_Pad1.05x0.95mm_HandSolder, symbol open-automation:C_1uF
- removed C?: C_10uF, Capacitor_SMD:C_0603_1608Metric_Pad1.05x0.95mm_HandSolder, symbol open-automation:C_10uF
- removed C?: C_0.1uF, Capacitor_SMD:C_0603_1608Metric_Pad1.05x0.95mm_HandSolder, symbol open-automation:C_0.1uF
- removed C?: C_100pF, Capacitor_SMD:C_0603_1608Metric_Pad1.05x0.95mm_HandSolder, symbol open-automation:C_100pF
- removed D? (x3): LED-0603-G, LED_SMD:LED_0603_1608Metric_Pad1.05x0.95mm_HandSolder, symbol open-automation:LED-0603-G
- removed D?: WS2812B, LED_SMD:LED_WS2812B_PLCC4_5.0x5.0mm_P3.2mm, symbol LED:WS2812B
- removed FACTORY?, PROG?, REBOOT?: SW_PUSH, Button_Switch_SMD:SW_SPST_KMR2, symbol liger-rescue:SW_PUSH
- removed J?: Conn_02x08_Odd_Even, Connector_PinHeader_2.54mm:PinHeader_2x08_P2.54mm_Vertical, symbol liger-rescue:Conn_02x08_Odd_Even
- removed R? (x3): R_1k, Resistor_SMD:R_0603_1608Metric_Pad1.05x0.95mm_HandSolder, symbol open-automation:R_1k
- removed R?: R_100k, Resistor_SMD:R_0603_1608Metric_Pad1.05x0.95mm_HandSolder, symbol liger-rescue:R_100k
- removed U?: ESP-WROOM-32, open-automation:ESP-WROOM-32, symbol liger-rescue:ESP-WROOM-32
- removed U?: soft-button-4x, open-automation:soft-button-4, symbol liger-rescue:soft-button-4x
- removed U?: housing-mounts, open-automation:generic-housing-mounts-md, symbol liger-rescue:housing-mounts-open-automation
- removed U?: PYQ2898, Package_TO_SOT_THT:TO-5-3, symbol open-automation:PYQ2898
- removed U?: AP2112, Package_TO_SOT_SMD:SOT-23-5_HandSoldering, symbol liger-rescue:AP2112
Connections:
- net labels removed: 3V3, BUTTON_LED, EN, FACTORY_RST, GND, I2S_BCLK, I2S_WS, PIR, PROG, RELAY_1, RELAY_2, RELAY_3, RELAY_4, RXD, TXD, T_DOWN, T_LEFT, T_RIGHT, T_UP, V_BAT, V_IN, V_USB, ZERO_DETECT
- wire segments 98 -> 0
Other:
- note removed: "ByPass CAPs"

Commit message: sent to boardhouse
Parts:
- added C1, C2: C_1uF, Capacitor_SMD:C_0603_1608Metric_Pad1.05x0.95mm_HandSolder, symbol open-automation:C_1uF
- added C3: C_0.1uF, Capacitor_SMD:C_0603_1608Metric_Pad1.05x0.95mm_HandSolder, symbol open-automation:C_0.1uF
- added J1: Conn_02x02_Odd_Even, Connector_PinHeader_2.54mm:PinHeader_2x02_P2.54mm_Vertical_SMD, symbol Connector_Generic:Conn_02x02_Odd_Even
- added P1: CONN_01X03, Connector_PinHeader_2.54mm:PinHeader_1x03_P2.54mm_Vertical, symbol open-automation:CONN_01X03
- added R1, R2, R3: R_10K, Resistor_SMD:R_0603_1608Metric_Pad1.05x0.95mm_HandSolder, symbol open-automation:R_10K
- added SW1: Rotary_Encoder_Switch, Rotary_Encoder:RotaryEncoder_Alps_EC11E-Switch_Vertical_H20mm, symbol open-automation:Rotary_Encoder_Switch
- added U1: AP2112, Package_TO_SOT_SMD:SOT-23-5_HandSoldering, symbol open-automation:AP2112
- added U2: PIR-DIGITAL, Package_TO_SOT_THT:TO-5-3, symbol open-automation:PIR-DIGITAL
Connections:
- new net 3V3: C2.1, C3.1, R1.2, R2.2, R3.2, U1.5 (VOUT), U2.1 (Vcc)
- new net 5V: C1.1, J1.1 (Pin_1), P1.1 (P1), U1.1 (Vin), U1.3 (EN)
- new net CLK_IO: R1.1, SW1.A
- new net DT_IO: R2.1, SW1.B
- new net GND: C1.2, C2.2, C3.2, J1.3 (Pin_3), P1.3 (P3), SW1.C, SW1.S2, U1.2 (GND), U2.3 (Vss)
- new net LED_IO: P1.2 (P2)
- new net PIR_IO: U2.2 (data)
- new net RXD: J1.4 (Pin_4)
- new net SW_IO: R3.1, SW1.S1
- new net TXD: J1.2 (Pin_2)
