File: circuits/microcontroller.sch (KiCad schematic (older format))
At the start: 0 parts

Commit message: init
Parts:
- added C18: C_10uF, Capacitor_SMD:C_0603_1608Metric_Pad1.05x0.95mm_HandSolder, symbol open-automation:C_10uF
- added C19: C_1uF, Capacitor_SMD:C_0603_1608Metric_Pad1.05x0.95mm_HandSolder, symbol open-automation:C_1uF
- added C20: C_0.1uF, Capacitor_SMD:C_0603_1608Metric_Pad1.05x0.95mm_HandSolder, symbol open-automation:C_0.1uF
- added D10, D11, D9: LED_G, Diode_SMD:D_0603_1608Metric_Pad1.05x0.95mm_HandSolder, symbol open-automation:LED_G
- added J7: Conn_02x05_Odd_Even, Connector_PinHeader_2.54mm:PinHeader_2x05_P2.54mm_Vertical, symbol open-automation:Conn_02x05_Odd_Even
- added R25, R26, R27, R28, R29, R30: R_10K, Resistor_SMD:R_0603_1608Metric_Pad1.05x0.95mm_HandSolder, symbol open-automation:R_10K
- added SW1, SW2, SW3: SW_PUSH, Button_Switch_SMD:SW_Push_1P1T_NO_CK_KMR2, symbol open-automation:SW_PUSH
- added U12: ESP-WROOM-32, open-automation:ESP-WROOM-32, symbol open-automation:ESP-WROOM-32
- added U13: SI7020-A20, open-automation:SI7020-A20, symbol open-automation:SI7020-A20
Connections:
- new net: R30.2, U12.24 (IO2)
- new net: D9.1 (K), R25.2
- new net: D10.1 (K), R26.2
- new net: D11.1 (K), R27.2
- new net 3V3: C18.1, C19.1, C20.1, D10.2 (A), D11.2 (A), D9.2 (A), R28.1, R29.1, U12.2 (3V3), U13.5 (Vin)
- new net ESP_EN: J7.7 (Pin_7), R25.1, SW1.1, U12.3 (EN)
- new net FACT: J7.5 (Pin_5), R27.1, SW3.1, U12.13 (IO14)
- new net GND: C18.2, C19.2, C20.2, J7.2 (Pin_2), J7.9 (Pin_9), R30.1, SW1.2, SW2.2, SW3.2, U12.1 (GND), U13.2 (GND)
- new net PROG: J7.3 (Pin_3), R26.1, SW2.1, U12.25 (IO0)
- new net RXD: J7.10 (Pin_10), U12.34 (RXD)
- new net SCL: J7.6 (Pin_6), R28.2, U12.33 (IO21), U13.6 (SCL)
- new net SDA: J7.4 (Pin_4), R29.2, U12.31 (IO19), U13.1 (SDA)
- new net SOFT_POWER: J7.1 (Pin_1)
- new net TXD: J7.8 (Pin_8), U12.35 (TXD)

Commit message: adding sheets
Parts:
- renumbered C18 to C?, C19 to C?, D9 to D?, D10 to D?, D11 to D?, R29 to R?, R28 to R?, R27 to R?, R26 to R?, R25 to R?, R30 to R?, U12 to U?
Changed lines of the file:
@@
 EESchema Schematic File Version 4
+LIBS:led-controller-cache
 EELAYER 29 0
 EELAYER END
 $Descr USLetter 11000 8500
 encoding utf-8
-Sheet 1 1
+Sheet 2 2
 Title ""
 Date ""
@@
 AR Path="/5CC0CE35" Ref="#PWR?"  Part="1"
 AR Path="/5A7BADDB/5CC0CE35" Ref="#PWR056"  Part="1"
-F 0 "#PWR056" H 6250 1850 50  0001 C CNN
+AR Path="/5D2CEC1B/5CC0CE35" Ref="#PWR?"  Part="1"
+F 0 "#PWR?" H 6250 1850 50  0001 C CNN
 F 1 "GND" H 6250 1950 50  0000 C CNN
 F 2 "" H 6250 2100 50  0000 C CNN
@@
 AR Path="/5CC0CE28" Ref="#PWR?"  Part="1"
 AR Path="/5A7BADDB/5CC0CE28" Ref="#PWR058"  Part="1"
-F 0 "#PWR058" H 6850 1400 50  0001 C CNN
+AR Path="/5D2CEC1B/5CC0CE28" Ref="#PWR?"  Part="1"
+F 0 "#PWR?" H 6850 1400 50  0001 C CNN
 F 1 "GND" V 6900 1500 50  0000 C CNN
 F 2 "" H 6850 1650 50  0000 C CNN
@@
 AR Path="/5CC0CE20" Ref="J?"  Part="1"
 AR Path="/5A7BADDB/5CC0CE20" Ref="J7"  Part="1"
-F 0 "J7" H 6550 2267 50  0000 C CNN
+AR Path="/5D2CEC1B/5CC0CE20" Ref="J?"  Part="1"
+F 0 "J?" H 6550 2267 50  0000 C CNN
 F 1 "Conn_02x05_Odd_Even" H 6550 2176 50  0000 C CNN
 F 2 "Connector_PinHeader_2.54mm:PinHeader_2x05_P2.54mm_Vertical" H 6500 1850 50  0001 C CNN
@@
 $EndComp
 $Comp
-L open-automation:GND #PWR052
+L open-automation:GND #PWR?
 U 1 1 5CC8CF13
 P 3100 2000
-F 0 "#PWR052" H 3100 1750 50  0001 C CNN
+F 0 "#PWR?" H 3100 1750 50  0001 C CNN
 F 1 "GND" H 3100 1850 50  0000 C CNN
 F 2 "" H 3100 2000 50  0000 C CNN
@@
 $EndComp
 $Comp
-L open-automation:GND #PWR054
+L open-automation:GND #PWR?
 U 1 1 5CC8C67A
 P 3400 2000
-F 0 "#PWR054" H 3400 1750 50  0001 C CNN
+F 0 "#PWR?" H 3400 1750 50  0001 C CNN
 F 1 "GND" H 3400 1850 50  0000 C CNN
 F 2 "" H 3400 2000 50  0000 C CNN
@@
 $EndComp
 $Comp
-L open-automation:GND #PWR055
+L open-automation:GND #PWR?
 U 1 1 59097974
 P 4550 3000
-F 0 "#PWR055" H 4550 2750 50  0001 C CNN
+F 0 "#PWR?" H 4550 2750 50  0001 C CNN
 F 1 "GND" H 4550 2850 50  0000 C CNN
 F 2 "" H 4550 3000 50  0000 C CNN
@@
 $EndComp
 $Comp
-L open-automation:ESP-WROOM-32 U12
+L open-automation:ESP-WROOM-32 U?
 U 1 1 5AFA4EFB
 P 5500 3700
-F 0 "U12" H 6100 2650 60  0000 C CNN
+F 0 "U?" H 6100 2650 60  0000 C CNN
 F 1 "ESP-WROOM-32" H 5500 4500 60  0000 C CNN
 F 2 "open-automation:ESP-WROOM-32" H 5150 4300 60  0001 C CNN
@@
 $EndComp
 $Comp
-L open-automation:GND #PWR053
+L open-automation:GND #PWR?
 U 1 1 5CC69861
 P 3200 4650
-F 0 "#PWR053" H 3200 4400 50  0001 C CNN
+F 0 "#PWR?" H 3200 4400 50  0001 C CNN
 F 1 "GND" H 3200 4500 50  0000 C CNN
 F 2 "" H 3200 4650 50  0000 C CNN
@@
 AR Path="/5ABD187E/5CC69855" Ref="SW?"  Part="1"
 AR Path="/5A7BADDB/5CC69855" Ref="SW3"  Part="1"
-F 0 "SW3" H 3200 4475 50  0000 C CNN
+AR Path="/5D2CEC1B/5CC69855" Ref="SW?"  Part="1"
+F 0 "SW?" H 3200 4475 50  0000 C CNN
 F 1 "SW_PUSH" H 3175 4200 50  0000 C CNN
 F 2 "Button_Switch_SMD:SW_Push_1P1T_NO_CK_KMR2" H 3200 4300 50  0001 C CNN
@@
 $EndComp
 $Comp
-L open-automation:GND #PWR051
+L open-automation:GND #PWR?
 U 1 1 5CC68123
 P 2650 4650
-F 0 "#PWR051" H 2650 4400 50  0001 C CNN
+F 0 "#PWR?" H 2650 4400 50  0001 C CNN
 F 1 "GND" H 2650 4500 50  0000 C CNN
 F 2 "" H 2650 4650 50  0000 C CNN
@@
 AR Path="/5ABD187E/5CC68117" Ref="SW?"  Part="1"
 AR Path="/5A7BADDB/5CC68117" Ref="SW2"  Part="1"
-F 0 "SW2" H 2650 4475 50  0000 C CNN
+AR Path="/5D2CEC1B/5CC68117" Ref="SW?"  Part="1"
+F 0 "SW?" H 2650 4475 50  0000 C CNN
 F 1 "SW_PUSH" H 2625 4200 50  0000 C CNN
 F 2 "Button_Switch_SMD:SW_Push_1P1T_NO_CK_KMR2" H 2650 4300 50  0001 C CNN
@@
 $EndComp
 $Comp
-L open-automation:GND #PWR050
+L open-automation:GND #PWR?
 U 1 1 5CC89C27
 P 2050 4650
-F 0 "#PWR050" H 2050 4400 50  0001 C CNN
+F 0 "#PWR?" H 2050 4400 50  0001 C CNN
 F 1 "GND" H 2050 4500 50  0000 C CNN
 F 2 "" H 2050 4650 50  0000 C CNN
@@
 AR Path="/5ABD187E/5CC89C1F" Ref="SW?"  Part="1"
 AR Path="/5A7BADDB/5CC89C1F" Ref="SW1"  Part="1"
-F 0 "SW1" H 2050 4475 50  0000 C CNN
+AR Path="/5D2CEC1B/5CC89C1F" Ref="SW?"  Part="1"
+F 0 "SW?" H 2050 4475 50  0000 C CNN
 F 1 "SW_PUSH" H 2025 4200 50  0000 C CNN
 F 2 "Button_Switch_SMD:SW_Push_1P1T_NO_CK_KMR2" H 2050 4300 50  0001 C CNN
@@
 AR Path="/5A8CA1FA/5CC805AD" Ref="C?"  Part="1"
 AR Path="/5A7BADDB/5CC805AD" Ref="C20"  Part="1"
-F 0 "C20" H 7400 3850 50  0000 L CNN
+AR Path="/5D2CEC1B/5CC805AD" Ref="C?"  Part="1"
+F 0 "C?" H 7400 3850 50  0000 L CNN
 F 1 "C_0.1uF" H 7350 3750 50  0000 L CNN
 F 2 "Capacitor_SMD:C_0603_1608Metric_Pad1.05x0.95mm_HandSolder" H 7750 4150 50  0001 C CNN
@@
 AR Path="/5A8CA1FA/5CC80592" Ref="U?"  Part="1"
 AR Path="/5A7BADDB/5CC80592" Ref="U13"  Part="1"
-F 0 "U13" H 8800 3900 60  0000 C CNN
+AR Path="/5D2CEC1B/5CC80592" Ref="U?"  Part="1"
+F 0 "U?" H 8800 3900 60  0000 C CNN
 F 1 "SI7020-A20" H 8600 4200 60  0000 C CNN
 F 2 "open-automation:SI7020-A20" H 8600 3700 60  0001 C CNN
@@
 AR Path="/5A8CA1FA/5CC80583" Ref="#PWR?"  Part="1"
 AR Path="/5A7BADDB/5CC80583" Ref="#PWR060"  Part="1"
-F 0 "#PWR060" H 8100 3800 50  0001 C CNN
+AR Path="/5D2CEC1B/5CC80583" Ref="#PWR?"  Part="1"
+F 0 "#PWR?" H 8100 3800 50  0001 C CNN
 F 1 "GND" H 8100 3900 50  0000 C CNN
 F 2 "" H 8100 4050 50  0000 C CNN
@@
 $EndComp
 $Comp
-L open-automation:C_1uF C19
+L open-automation:C_1uF C?
 U 1 1 5B2CA474
 P 3400 1800
-F 0 "C19" H 3500 1800 50  0000 L CNN
+F 0 "C?" H 3500 1800 50  0000 L CNN
 F 1 "C_1uF" H 3400 1700 50  0000 L CNN
 F 2 "Capacitor_SMD:C_0603_1608Metric_Pad1.05x0.95mm_HandSolder" H 3500 2100 50  0001 C CNN
@@
 $EndComp
 $Comp
-L open-automation:C_10uF C18
+L open-automation:C_10uF C?
 U 1 1 5B2706A8
 P 3100 1800
-F 0 "C18" H 2850 1800 50  0000 L CNN
+F 0 "C?" H 2850 1800 50  0000 L CNN
 F 1 "C_10uF" H 2800 1700 50  0000 L CNN
 F 2 "Capacitor_SMD:C_0603_1608Metric_Pad1.05x0.95mm_HandSolder" H 3200 2100 50  0001 C CNN
@@
 $EndComp
 $Comp
-L open-automation:GND #PWR057
+L open-automation:GND #PWR?
 U 1 1 5AF61DA0
 P 6350 4950
-F 0 "#PWR057" H 6350 4700 50  0001 C CNN
+F 0 "#PWR?" H 6350 4700 50  0001 C CNN
 F 1 "GND" H 6350 4800 50  0000 C CNN
 F 2 "" H 6350 4950 50  0000 C CNN
@@
 $EndComp
 $Comp
-L open-automation:R_10K R29
+L open-automation:R_10K R?
 U 1 1 5CC267DD
 P 4300 1950
-F 0 "R29" V 4300 1950 50  0000 C CNN
+F 0 "R?" V 4300 1950 50  0000 C CNN
 F 1 "R_10K" V 4400 1950 50  0000 C CNN
 F 2 "Resistor_SMD:R_0603_1608Metric_Pad1.05x0.95mm_HandSolder" V 4230 1950 50  0001 C CNN
@@
 $EndComp
 $Comp
-L open-automation:R_10K R28
+L open-automation:R_10K R?
 U 1 1 5CC28727
 P 4300 1800
-F 0 "R28" V 4300 1800 50  0000 C CNN
+F 0 "R?" V 4300 1800 50  0000 C CNN
 F 1 "R_10K" V 4184 1800 50  0000 C CNN
 F 2 "Resistor_SMD:R_0603_1608Metric_Pad1.05x0.95mm_HandSolder" V 4230 1800 50  0001 C CNN
@@
 $EndComp
 $Comp
-L open-automation:R_10K R27
+L open-automation:R_10K R?
 U 1 1 5CC2B523
 P 3200 3700
-F 0 "R27" V 2993 3700 50  0000 C CNN
+F 0 "R?" V 2993 3700 50  0000 C CNN
 F 1 "R_10K" V 3084 3700 50  0000 C CNN
 F 2 "Resistor_SMD:R_0603_1608Metric_Pad1.05x0.95mm_HandSolder" V 3130 3700 50  0001 C CNN
@@
 $EndComp
 $Comp
-L open-automation:R_10K R26
+L open-automation:R_10K R?
 U 1 1 5CC2D1AD
 P 2650 3700
-F 0 "R26" V 2443 3700 50  0000 C CNN
+F 0 "R?" V 2443 3700 50  0000 C CNN
 F 1 "R_10K" V 2534 3700 50  0000 C CNN
 F 2 "Resistor_SMD:R_0603_1608Metric_Pad1.05x0.95mm_HandSolder" V 2580 3700 50  0001 C CNN
@@
 $EndComp
 $Comp
-L open-automation:R_10K R25
+L open-automation:R_10K R?
 U 1 1 5CC2EC19
 P 2050 3700
-F 0 "R25" V 1843 3700 50  0000 C CNN
+F 0 "R?" V 1843 3700 50  0000 C CNN
 F 1 "R_10K" V 1934 3700 50  0000 C CNN
 F 2 "Resistor_SMD:R_0603_1608Metric_Pad1.05x0.95mm_HandSolder" V 1980 3700 50  0001 C CNN
@@
 $EndComp
 $Comp
-L open-automation:R_10K R30
+L open-automation:R_10K R?
 U 1 1 5CC3139A
 P 6100 4950
-F 0 "R30" V 5893 4950 50  0000 C CNN
+F 0 "R?" V 5893 4950 50  0000 C CNN
 F 1 "R_10K" V 5984 4950 50  0000 C CNN
 F 2 "Resistor_SMD:R_0603_1608Metric_Pad1.05x0.95mm_HandSolder" V 6030 4950 50  0001 C CNN
@@
 $EndComp
 $Comp
-L open-automation:LED_G D9
+L open-automation:LED_G D?
 U 1 1 5CC255BE
 P 2050 3300
-F 0 "D9" V 2089 3183 50  0000 R CNN
+F 0 "D?" V 2089 3183 50  0000 R CNN
 F 1 "LED_G" V 1998 3183 50  0000 R CNN
 F 2 "Diode_SMD:D_0603_1608Metric_Pad1.05x0.95mm_HandSolder" H 2050 3300 50  0001 C CNN
@@
 $EndComp
 $Comp
-L open-automation:LED_G D10
+L open-automation:LED_G D?
 U 1 1 5CC26ACF
 P 2650 3300
-F 0 "D10" V 2689 3183 50  0000 R CNN
+F 0 "D?" V 2689 3183 50  0000 R CNN
 F 1 "LED_G" V 2598 3183 50  0000 R CNN
 F 2 "Diode_SMD:D_0603_1608Metric_Pad1.05x0.95mm_HandSolder" H 2650 3300 50  0001 C CNN
@@
 $EndComp
 $Comp
-L open-automation:LED_G D11
+L open-automation:LED_G D?
 U 1 1 5CC27619
 P 3200 3300
-F 0 "D11" V 3239 3183 50  0000 R CNN
+F 0 "D?" V 3239 3183 50  0000 R CNN
 F 1 "LED_G" V 3148 3183 50  0000 R CNN
 F 2 "Diode_SMD:D_0603_1608Metric_Pad1.05x0.95mm_HandSolder" H 3200 3300 50  0001 C CNN
@@
 AR Path="/5A8CA1FA/5CCAE63E" Ref="#PWR?"  Part="1"
 AR Path="/5A7BADDB/5CCAE63E" Ref="#PWR0103"  Part="1"
-F 0 "#PWR0103" H 7650 3800 50  0001 C CNN
+AR Path="/5D2CEC1B/5CCAE63E" Ref="#PWR?"  Part="1"
+F 0 "#PWR?" H 7650 3800 50  0001 C CNN
 F 1 "GND" H 7650 3900 50  0000 C CNN
 F 2 "" H 7650 4050 50  0000 C CNN

Commit message: sent to boardhouse
Parts:
- removed J7: Conn_02x05_Odd_Even, Connector_PinHeader_2.54mm:PinHeader_2x05_P2.54mm_Vertical, symbol open-automation:Conn_02x05_Odd_Even
- added J2: Conn_02x07_Odd_Even, Connector_PinHeader_2.54mm:PinHeader_2x07_P2.54mm_Vertical_SMD, symbol Connector_Generic:Conn_02x07_Odd_Even
- gave numbers to parts that had none: 12
- renumbered C20 to C6, SW1 to SW2, SW2 to SW3, SW3 to SW4, U13 to U4
Connections:
- net 3V3: now also J2.11 (Pin_11)
- net FACT: now also J2.5 (Pin_5)
- net GND: now also J2.13 (Pin_13), J2.14 (Pin_14)
- net SCL: now also J2.8 (Pin_8)
- net SDA: now also J2.10 (Pin_10)
- net IO25: now reaches U3.10 (IO25)
- net IO25: now also J2.4 (Pin_4)
- net IO26: now reaches U3.11 (IO26)
- net IO26: now also J2.6 (Pin_6)
- net IO27: now reaches U3.12 (IO27)
- net IO12: now reaches U3.14 (IO12)
- net IO12: now also J2.1 (Pin_1)
- net IO13: now reaches U3.16 (IO13)
- net IO13: now also J2.3 (Pin_3)
- net IO4: now reaches U3.26 (IO4)
- net IO16: now reaches U3.27 (IO16)
- net IO17: now reaches U3.28 (IO17)
- net IO5: now reaches U3.29 (IO5)
- net IO18: now reaches U3.30 (IO18)
- net IO22: now reaches U3.36 (IO22)
- net IO22: now also J2.9 (Pin_9)
- net IO23: now reaches U3.37 (IO23)
- net IO23: now also J2.7 (Pin_7)
- net IO34: now reaches U3.6 (IO34)
- net IO35: now reaches U3.7 (IO35)
- net IO32: now reaches U3.8 (IO32)
- net IO33: now reaches U3.9 (IO33)
- net IO33: now also J2.2 (Pin_2)
- net ESP_EN renamed EN
- new net 5V: J2.12 (Pin_12)
